Commit message: Update ros2_control.xacro

File: cloud_robot/urdf/ros2_control.xacro (robot description, xacro)
@@ -0,0 +1,43 @@
+<ros2_control name="DiffDriveSystem" type="system">
+  <hardware>
+    <plugin>cloud_hardware/DiffDriveHW</plugin>
+    <!-- LEFT TRACK -->
+    <param name="left.name">left_track</param>
+    <param name="left.slp_gpio">22</param>
+    <param name="left.dir_gpio">24</param>
+    <param name="left.pwm_gpio">12</param>
+    <param name="left.rpm_motor">220.0</param>
+    <param name="left.gear_ratio">1.73</param>
+    <param name="left.max_accel">16.0</param>
+    <param name="left.invert_direction">true</param>
+    <!-- RIGHT TRACK -->
+    <param name="right.name">right_track</param>
+    <param name="right.slp_gpio">23</param>
+    <param name="right.dir_gpio">25</param>
+    <param name="right.pwm_gpio">13</param>
+    <param name="right.rpm_motor">220.0</param>
+    <param name="right.gear_ratio">1.73</param>
+    <param name="right.max_accel">16.0</param>
+    <param name="right.invert_direction">true</param>
+  </hardware>
+  <joint name="Left_Front_Wheel_1">
+    <command_interface name="velocity"/>
+    <state_interface name="velocity"/>
+    <state_interface name="position"/>
+  </joint>
+  <joint name="Right_Front_Wheel_1">
+    <command_interface name="velocity"/>
+    <state_interface name="velocity"/>
+    <state_interface name="position"/>
+  </joint>
+  <joint name="Left_Rear_Wheel_1">
+    <command_interface name="velocity"/>
+    <state_interface name="velocity"/>
+    <state_interface name="position"/>
+  </joint>
+  <joint name="left_track_joint">
+    <command_interface name="velocity"/>
+    <state_interface name="velocity"/>
+    <state_interface name="position"/>
+  </joint>
+</ros2_control>

Commit message: Update ros2_control.xacro

File: cloud_robot/urdf/ros2_control.xacro (robot description, xacro)
@@ -42,2 +42,130 @@
   </joint>
 </ros2_control>
+<ros2_control name="ServoHW" type="system">
+  <hardware>
+    <plugin>cloud_hardware/ServoHW</plugin>
+  </hardware>
+  <!-- FLIPPERS -->
+  <joint name="Left_Front_Fliper_1">
+    <command_interface name="position"/>
+    <state_interface name="position"/>
+    <param name="channel">0</param>
+    <param name="rad_min">-2.35</param>
+    <param name="rad_max">2.35</param>
+    <param name="us_min">500</param>
+    <param name="us_max">2500</param>
+    <param name="zero_offset_rad">2.35</param>
+    <param name="invert">false</param>
+  </joint>
+  <joint name="Right_Front_Fliper_1">
+    <command_interface name="position"/>
+    <state_interface name="position"/>
+    <param name="channel">1</param>
+    <param name="rad_min">-2.35</param>
+    <param name="rad_max">2.35</param>
+    <param name="us_min">500</param>
+    <param name="us_max">2500</param>
+    <param name="zero_offset_rad">2.35</param>
+    <param name="invert">true</param>
+  </joint>
+  <joint name="Left_Rear_Fliper_1">
+    <command_interface name="position"/>
+    <state_interface name="position"/>
+    <param name="channel">2</param>
+    <param name="rad_min">-2.35</param>
+    <param name="rad_max">2.35</param>
+    <param name="us_min">500</param>
+    <param name="us_max">2500</param>
+    <param name="zero_offset_rad">2.35</param>
+    <param name="invert">true</param>
+  </joint>
+  <joint name="Right_Rear_Wheel_1">
+    <command_interface name="position"/>
+    <state_interface name="position"/>
+    <param name="channel">3</param>
+    <param name="rad_min">-2.35</param>
+    <param name="rad_max">2.35</param>
+    <param name="us_min">500</param>
+    <param name="us_max">2500</param>
+    <param name="zero_offset_rad">2.35</param>
+    <param name="invert">false</param>
+  </joint>
+  <!-- ARM -->
+  <joint name="Joint_1_1">
+    <command_interface name="position"/>
+    <state_interface name="position"/>
+    <param name="channel">4</param>
+    <param name="rad_min">-2.35</param>
+    <param name="rad_max">2.35</param>
+    <param name="us_min">500</param>
+    <param name="us_max">2500</param>
+    <param name="zero_offset_rad">2.35</param>
+    <param name="invert">false</param>
+  </joint>
+  <joint name="Joint_Bridge_1_1">
+    <command_interface name="position"/>
+    <state_interface name="position"/>
+    <param name="channel">5</param>
+    <param name="rad_min">-2.35</param>
+    <param name="rad_max">2.35</param>
+    <param name="us_min">500</param>
+    <param name="us_max">2500</param>
+    <param name="zero_offset_rad">2.35</param>
+    <param name="invert">false</param>
+  </joint>
+  <joint name="Joint_Bridge_2_1">
+    <command_interface name="position"/>
+    <state_interface name="position"/>
+    <param name="channel">6</param>
+    <param name="rad_min">-2.35</param>
+    <param name="rad_max">2.35</param>
+    <param name="us_min">500</param>
+    <param name="us_max">2500</param>
+    <param name="zero_offset_rad">2.35</param>
+    <param name="invert">false</param>
+  </joint>
+  <joint name="Joint_2_1">
+    <command_interface name="position"/>
+    <state_interface name="position"/>
+    <param name="channel">7</param>
+    <param name="rad_min">-2.35</param>
+    <param name="rad_max">2.35</param>
+    <param name="us_min">500</param>
+    <param name="us_max">2500</param>
+    <param name="zero_offset_rad">2.35</param>
+    <param name="invert">false</param>
+  </joint>
+  <joint name="Joint_3_1">
+    <command_interface name="position"/>
+    <state_interface name="position"/>
+    <param name="channel">8</param>
+    <param name="rad_min">-2.35</param>
+    <param name="rad_max">2.35</param>
+    <param name="us_min">500</param>
+    <param name="us_max">2500</param>
+    <param name="zero_offset_rad">2.35</param>
+    <param name="invert">false</param>
+  </joint>
+  <joint name="Joint_4_1">
+    <command_interface name="position"/>
+    <state_interface name="position"/>
+    <param name="channel">9</param>
+    <param name="rad_min">-2.35</param>
+    <param name="rad_max">2.35</param>
+    <param name="us_min">500</param>
+    <param name="us_max">2500</param>
+    <param name="zero_offset_rad">2.35</param>
+    <param name="invert">false</param>
+  </joint>
+  <joint name="Joint_5_1">
+    <command_interface name="position"/>
+    <state_interface name="position"/>
+    <param name="channel">10</param>
+    <param name="rad_min">-2.35</param>
+    <param name="rad_max">2.35</param>
+    <param name="us_min">500</param>
+    <param name="us_max">2500</param>
+    <param name="zero_offset_rad">2.35</param>
+    <param name="invert">false</param>
+  </joint>
+</ros2_control>

Commit message: Update ros2_control.xacro

File: cloud_robot/urdf/ros2_control.xacro (robot description, xacro)
@@ -1,7 +1,7 @@
+<?xml version="1.0" ?>
+<robot name="URDF_DIRECCION_X" xmlns:xacro="http://www.ros.org/wiki/xacro" >
 <ros2_control name="DiffDriveSystem" type="system">
   <hardware>
-    <plugin>cloud_hardware/DiffDriveHW</plugin>
-    <!-- LEFT TRACK -->
-    <param name="left.name">left_track</param>
+    <plugin>cloud_robot/DiffDriveHW</plugin>
     <param name="left.slp_gpio">22</param>
     <param name="left.dir_gpio">24</param>
@@ -9,8 +9,6 @@
     <param name="left.rpm_motor">220.0</param>
     <param name="left.gear_ratio">1.73</param>
-    <param name="left.max_accel">16.0</param>
-    <param name="left.invert_direction">true</param>
-    <!-- RIGHT TRACK -->
-    <param name="right.name">right_track</param>
+    <param name="left.max_accel">25.0</param>
+    <param name="left.invert_direction">false</param>
     <param name="right.slp_gpio">23</param>
     <param name="right.dir_gpio">25</param>
@@ -18,23 +16,24 @@
     <param name="right.rpm_motor">220.0</param>
     <param name="right.gear_ratio">1.73</param>
-    <param name="right.max_accel">16.0</param>
+    <param name="right.max_accel">25.0</param>
     <param name="right.invert_direction">true</param>
   </hardware>
-  <joint name="Left_Front_Wheel_1">
+  <!-- Joints -->
+  <joint name="Revolucion_1">  <!-- left front wheel -->
     <command_interface name="velocity"/>
     <state_interface name="velocity"/>
     <state_interface name="position"/>
   </joint>
-  <joint name="Right_Front_Wheel_1">
+  <joint name="Revolucion_2">  <!-- right front wheel -->
     <command_interface name="velocity"/>
     <state_interface name="velocity"/>
     <state_interface name="position"/>
   </joint>
-  <joint name="Left_Rear_Wheel_1">
+  <joint name="Revolucion_3">  <!-- left rear wheel -->
     <command_interface name="velocity"/>
     <state_interface name="velocity"/>
     <state_interface name="position"/>
   </joint>
-  <joint name="left_track_joint">
+  <joint name="Revolucion_4">  <!--  right rear wheel -->
     <command_interface name="velocity"/>
     <state_interface name="velocity"/>
@@ -44,8 +43,8 @@
 <ros2_control name="ServoHW" type="system">
   <hardware>
-    <plugin>cloud_hardware/ServoHW</plugin>
+    <plugin>cloud_robot/ServoHW</plugin>
   </hardware>
   <!-- FLIPPERS -->
-  <joint name="Left_Front_Fliper_1">
+  <joint name="Revolucion_5">  <!--  left front flipper -->
     <command_interface name="position"/>
     <state_interface name="position"/>
@@ -56,7 +55,7 @@
     <param name="us_max">2500</param>
     <param name="zero_offset_rad">2.35</param>
-    <param name="invert">false</param>
+    <param name="invert">true</param>
   </joint>
-  <joint name="Right_Front_Fliper_1">
+  <joint name="Revolucion_6">  <!--  right front flipper -->
     <command_interface name="position"/>
     <state_interface name="position"/>
@@ -67,7 +66,7 @@
     <param name="us_max">2500</param>
     <param name="zero_offset_rad">2.35</param>
-    <param name="invert">true</param>
+    <param name="invert">false</param>
   </joint>
-  <joint name="Left_Rear_Fliper_1">
+  <joint name="Revolucion_7">  <!--  right rear flipper -->
     <command_interface name="position"/>
     <state_interface name="position"/>
@@ -80,5 +79,5 @@
     <param name="invert">true</param>
   </joint>
-  <joint name="Right_Rear_Wheel_1">
+  <joint name="Revolucion_8">  <!--  left rear flipper -->
     <command_interface name="position"/>
     <state_interface name="position"/>
@@ -92,5 +91,5 @@
   </joint>
   <!-- ARM -->
-  <joint name="Joint_1_1">
+  <joint name="Revolucion_9">  <!--  base to joint 1 -->
     <command_interface name="position"/>
     <state_interface name="position"/>
@@ -103,38 +102,38 @@
     <param name="invert">false</param>
   </joint>
-  <joint name="Joint_Bridge_1_1">
+  <joint name="Revolucion_10"> <!--  joint 1 to joint bridge 1 -->
     <command_interface name="position"/>
     <state_interface name="position"/>
     <param name="channel">5</param>
-    <param name="rad_min">-2.35</param>
-    <param name="rad_max">2.35</param>
-    <param name="us_min">500</param>
-    <param name="us_max">2500</param>
-    <param name="zero_offset_rad">2.35</param>
+    <param name="rad_min">0</param>
+    <param name="rad_max">2.70</param>
+    <param name="us_min">873</param>
+    <param name="us_max">2000</param>
+    <param name="zero_offset_rad">0</param>
     <param name="invert">false</param>
   </joint>
-  <joint name="Joint_Bridge_2_1">
+  <joint name="Revolucion_11"> <!--  joint 1 to joint bridge 2 -->
+    <command_interface name="position"/>
+    <state_interface name="position"/>
+    <param name="channel">12</param>
+    <param name="rad_min">0</param>
+    <param name="rad_max">2.70</param>
+    <param name="us_min">873</param>
+    <param name="us_max">2000</param>
+    <param name="zero_offset_rad">0</param>
+    <param name="invert">false</param>
+  </joint>
+  <joint name="Revolucion_12">  <!--  joint bridge 2 to joint 2-->
     <command_interface name="position"/>
     <state_interface name="position"/>
     <param name="channel">6</param>
-    <param name="rad_min">-2.35</param>
-    <param name="rad_max">2.35</param>
+    <param name="rad_min">0</param>
+    <param name="rad_max">3.14</param>
     <param name="us_min">500</param>
-    <param name="us_max">2500</param>
-    <param name="zero_offset_rad">2.35</param>
+    <param name="us_max">1600</param>
+    <param name="zero_offset_rad">0</param>
     <param name="invert">false</param>
   </joint>
-  <joint name="Joint_2_1">
-    <command_interface name="position"/>
-    <state_interface name="position"/>
-    <param name="channel">7</param>
-    <param name="rad_min">-2.35</param>
-    <param name="rad_max">2.35</param>
-    <param name="us_min">500</param>
-    <param name="us_max">2500</param>
-    <param name="zero_offset_rad">2.35</param>
-    <param name="invert">false</param>
-  </joint>
-  <joint name="Joint_3_1">
+  <joint name="Revolucion_13"> <!--  joint 2 to  joint 3-->
     <command_interface name="position"/>
     <state_interface name="position"/>
@@ -147,5 +146,5 @@
     <param name="invert">false</param>
   </joint>
-  <joint name="Joint_4_1">
+  <joint name="Revolucion_14"> <!--  joint 3 to  joint 4-->
     <command_interface name="position"/>
     <state_interface name="position"/>
@@ -158,5 +157,5 @@
     <param name="invert">false</param>
   </joint>
-  <joint name="Joint_5_1">
+  <joint name="Revolucion_15">  <!--  joint 4 to  joint 5-->
     <command_interface name="position"/>
     <state_interface name="position"/>
@@ -170,2 +169,3 @@
   </joint>
 </ros2_control>
+</robot>
